Commit message: update model

File: handrobot_model/hand_robot.urdf (robot description, URDF)
Before this commit: robot hand_robot, 60 links, 59 joints
Links:
- link base_link: mass 0.274553101575067 -> 0.616402354567036; geometry collision mesh filename=package://palm_ver2/meshes/base_link.stl; visual mesh filename=package://palm_ver2/meshes/base_link.dae
- link dummy_link1: mass 0.0119886897783525 -> 0.00131295075943631; geometry collision mesh filename=package://palm_ver2/meshes/dummy_link1.stl; visual mesh filename=package://palm_ver2/meshes/dummy_link1.dae
- link dummy_link2: mass 0.0119886897783526 -> 0.00131295075943631; geometry collision mesh filename=package://palm_ver2/meshes/dummy_link2.stl; visual mesh filename=package://palm_ver2/meshes/dummy_link2.dae
- link dummy_link3: mass 0.0119886897783526 -> 0.00131295075943631; geometry collision mesh filename=package://palm_ver2/meshes/dummy_link3.stl; visual mesh filename=package://palm_ver2/meshes/dummy_link3.dae
- link dummy_link4: mass 0.0119886897783526 -> 0.00131295075943631; geometry collision mesh filename=package://palm_ver2/meshes/dummy_link4.stl; visual mesh filename=package://palm_ver2/meshes/dummy_link4.dae
- link dummy_link5: mass 0.0119886601362974 -> 0.0013129474786583; geometry collision mesh filename=package://palm_ver2/meshes/dummy_link5.stl; visual mesh filename=package://palm_ver2/meshes/dummy_link5.dae
- link index_module4_base_link: mass 0.0143355339373342 -> 0.015; geometry collision mesh filename=package://fingertip_ver2/meshes/base_link.stl; visual mesh filename=package://fingertip_ver2/meshes/base_link.dae
- link little_module4_base_link: mass 0.0143355339373342 -> 0.015; geometry collision mesh filename=package://fingertip_ver2/meshes/base_link.stl; visual mesh filename=package://fingertip_ver2/meshes/base_link.dae
- link middle_module4_base_link: mass 0.0143355339373342 -> 0.015; geometry collision mesh filename=package://fingertip_ver2/meshes/base_link.stl; visual mesh filename=package://fingertip_ver2/meshes/base_link.dae
- link ring_module4_base_link: mass 0.0143355339373342 -> 0.015; geometry collision mesh filename=package://fingertip_ver2/meshes/base_link.stl; visual mesh filename=package://fingertip_ver2/meshes/base_link.dae
- link thumb_module4_base_link: mass 0.0143355339373342 -> 0.015; geometry collision mesh filename=package://fingertip_ver2/meshes/base_link.stl; visual mesh filename=package://fingertip_ver2/meshes/base_link.dae
Joints:
- joint dummy_joint1: origin xyz=-0.134 0.0 0.104 rpy=0.0 -0.0 0.0 -> xyz=0.0114999999999997 0.0569905394079266 0.147 rpy=0.0 -0.0 -1.5707963267949003
- joint dummy_joint2: origin xyz=-0.0790000000000001 0.0 0.148 rpy=0.0 -0.0 0.0 -> xyz=0.0114999999999993 0.00199053940792622 0.191 rpy=-0.0 -0.0 -1.57079632679489
- joint dummy_joint3: origin xyz=-0.024 0.0 0.169 rpy=0.0 -0.0 0.0 -> xyz=0.0114999999999994 -0.0530094605920739 0.212 rpy=-0.0 -0.0 -1.57079632679489
- joint dummy_joint4: origin xyz=0.0309999999999999 0.0 0.138 rpy=0.0 -0.0 0.0 -> xyz=0.011499999999999 -0.108009460592074 0.181 rpy=-0.0 -0.0 -1.57079632679489
- joint dummy_joint5: origin xyz=0.018463196704848 0.0 0.0524638930461059 rpy=3.14159265358979 0.6356359574700541 3.14159265358978 -> xyz=0.0114999999999986 -0.0954726572969222 0.0954638930461058 rpy=3.14159265358979 0.6356359574700541 1.57079632679489

File: handrobot_model/hand_robot.xacro (robot description, xacro)
@@ -1,15 +1,15 @@
 <robot name="hand_robot" xmlns:xacro="http://ros.org/wiki/xacro">
   <xacro:include filename="$(find screw_cross_module_cover_invert_50mm)/urdf/screw_cross_module_cover_invert_50mm_dae.xacro" />
-  <xacro:include filename="$(find palm)/urdf/palm_dae.xacro" />
-  <xacro:include filename="$(find fingertip)/urdf/fingertip_dae.xacro" />
+  <xacro:include filename="$(find palm_ver2)/urdf/palm_ver2_dae.xacro" />
+  <xacro:include filename="$(find fingertip_ver2)/urdf/fingertip_ver2_dae.xacro" />
   <xacro:include filename="$(find screw_cm_module)/urdf/screw_cm_module_dae.xacro" />
   <xacro:include filename="$(find screw_26mmhinge_module_cover_40deg)/urdf/screw_26mmhinge_module_cover_40deg_dae.xacro" />
   <xacro:include filename="$(find screw_26mmhinge_module_cover_0deg)/urdf/screw_26mmhinge_module_cover_0deg_dae.xacro" />
   <link name="world" />
-  <xacro:palm
+  <xacro:palm_ver2
     prefix=""
     parent_link="world">
     <origin xyz="0 0 0" rpy="0 0 0"/>
-  </xacro:palm>
+  </xacro:palm_ver2>
   <xacro:screw_cross_module_cover_invert_50mm
     prefix="little_module1_"
@@ -27,9 +27,9 @@
     rpy="0 0 1.5707963267948966">
   </xacro:screw_26mmhinge_module_cover_40deg>
-  <xacro:fingertip
+  <xacro:fingertip_ver2
     prefix="little_module4_"
     parent_link="little_module3_dummy_link"
     rpy="0 0 1.5707963267948966">
-  </xacro:fingertip>
+  </xacro:fingertip_ver2>
   <xacro:screw_cross_module_cover_invert_50mm
     prefix="ring_module1_"
@@ -47,9 +47,9 @@
     rpy="0 0 1.5707963267948966">
   </xacro:screw_26mmhinge_module_cover_40deg>
-  <xacro:fingertip
+  <xacro:fingertip_ver2
     prefix="ring_module4_"
     parent_link="ring_module3_dummy_link"
     rpy="0 0 1.5707963267948966">
-  </xacro:fingertip>
+  </xacro:fingertip_ver2>
   <xacro:screw_cross_module_cover_invert_50mm
     prefix="middle_module1_"
@@ -67,9 +67,9 @@
     rpy="0 0 1.5707963267948966">
   </xacro:screw_26mmhinge_module_cover_40deg>
-  <xacro:fingertip
+  <xacro:fingertip_ver2
     prefix="middle_module4_"
     parent_link="middle_module3_dummy_link"
     rpy="0 0 1.5707963267948966">
-  </xacro:fingertip>
+  </xacro:fingertip_ver2>
   <xacro:screw_cross_module_cover_invert_50mm
     prefix="index_module1_"
@@ -87,9 +87,9 @@
     rpy="0 0 1.5707963267948966">
   </xacro:screw_26mmhinge_module_cover_40deg>
-  <xacro:fingertip
+  <xacro:fingertip_ver2
     prefix="index_module4_"
     parent_link="index_module3_dummy_link"
     rpy="0 0 1.5707963267948966">
-  </xacro:fingertip>
+  </xacro:fingertip_ver2>
   <xacro:screw_cm_module
     prefix="thumb_module1_"
@@ -107,8 +107,8 @@
     rpy="0 0 1.5707963267948966">
   </xacro:screw_26mmhinge_module_cover_40deg>
-  <xacro:fingertip
+  <xacro:fingertip_ver2
     prefix="thumb_module4_"
     parent_link="thumb_module3_dummy_link"
     rpy="0 0 1.5707963267948966">
-  </xacro:fingertip>
+  </xacro:fingertip_ver2>
 </robot>
